Commit message: doosanH2515 and slider

File: awi_description/urdf/cart_with_h2515.urdf.xacro (robot description, xacro)
@@ -53,9 +53,9 @@
     <parent link="slideBar"/>
     <child link="cart"/>
-    <limit effort="10000.0" lower="-15.0" upper="15.0" velocity="0.25"/>
-    <dynamics damping="50.0" friction="10.0"/>
+    <limit effort="10000.0" lower="-15.0" upper="15.0" velocity="2.0"/>
+    <dynamics damping="5.0" friction="1.0"/>
   </joint>
   <!-- 2. DOOSAN H2515 GÖVDESİ -->
-  <xacro:include filename="$(find dsr_description2)/xacro/macro.h2515.blue.xacro" />
+  <xacro:include filename="$(find awi_description)/xacro/macro.h2515.blue.xacro" />
   <xacro:h2515 namespace="$(arg namespace)"/>
   <!-- 3. KART MONTAJI -->
@@ -70,5 +70,5 @@
   <!-- 5. TEK GAZEBO ROS2 CONTROL PLUGIN -->
   <gazebo>
-    <plugin filename="gz_ros2_control-system" name="gz_ros2_control::GazeboSimROS2ControlPlugin">
+    <plugin filename="ign_ros2_control-system" name="ign_ros2_control::IgnitionROS2ControlPlugin">
       <parameters>$(find awi_description)/config/cell_controllers.yaml</parameters>
     </plugin>

File: awi_description/urdf/inspection_cell_ros2_control.xacro (robot description, xacro)
@@ -5,8 +5,7 @@
       <hardware>
         <xacro:if value="${sim_mode}">
-          <plugin>gz_ros2_control/GazeboSimSystem</plugin>
+          <plugin>ign_ros2_control/IgnitionSystem</plugin>
         </xacro:if>
         <xacro:unless value="${sim_mode}">
-          <!-- Gerçek donanıma geçildiğinde Doosan veya hibrit sürücü eklentisi -->
           <plugin>dsr_hardware2/DRHWInterface</plugin>
           <param name="host">192.168.1.100</param>
@@ -17,83 +16,38 @@
         </xacro:unless>
       </hardware>
-      <!-- 1. KIZAK EKLEMİ (Linear Axis) -->
+      <!-- 1. KIZAK EKLEMİ -->
       <joint name="slider_to_cart">
         <command_interface name="position">
-          <param name="min">-15</param>
-          <param name="max">15</param>
+          <param name="min">-15.0</param>
+          <param name="max">15.0</param>
         </command_interface>
         <state_interface name="position">
           <param name="initial_value">0.0</param>
         </state_interface>
-        <state_interface name="velocity"/>
-        <state_interface name="effort"/>
-      </joint>
-      <!-- 2. DOOSAN H2515 EKLEMLERİ (1'den 6'ya) -->
-      <joint name="joint_1">
-        <command_interface name="position">
-          <param name="min">{-2*pi}</param>
-          <param name="max">{2*pi}</param>
-        </command_interface>
-        <command_interface name="velocity"/>
-        <state_interface name="position">
+        <state_interface name="velocity">
           <param name="initial_value">0.0</param>
         </state_interface>
-        <state_interface name="velocity"/>
       </joint>
-      <joint name="joint_2">
-        <command_interface name="position">
-          <param name="min">{-2*pi}</param>
-          <param name="max">{2*pi}</param>
-        </command_interface>
-        <command_interface name="velocity"/>
-        <state_interface name="position">
-          <param name="initial_value">0.0</param>
-        </state_interface>
-        <state_interface name="velocity"/>
-      </joint>
-      <joint name="joint_3">
-        <command_interface name="position">
-          <param name="min">{-pi}</param>
-          <param name="max">{pi}</param>
-        </command_interface>
-        <command_interface name="velocity"/>
-        <state_interface name="position">
-          <param name="initial_value">0.0</param>
-        </state_interface>
-        <state_interface name="velocity"/>
-      </joint>
-      <joint name="joint_4">
-        <command_interface name="position">
-          <param name="min">{-2*pi}</param>
-          <param name="max">{2*pi}</param>
-        </command_interface>
-        <command_interface name="velocity"/>
-        <state_interface name="position">
-          <param name="initial_value">0.0</param>
-        </state_interface>
-        <state_interface name="velocity"/>
-      </joint>
-      <joint name="joint_5">
-        <command_interface name="position">
-          <param name="min">{-2*pi}</param>
-          <param name="max">{2*pi}</param>
-        </command_interface>
-        <command_interface name="velocity"/>
-        <state_interface name="position">
-          <param name="initial_value">0.0</param>
-        </state_interface>
-        <state_interface name="velocity"/>
-      </joint>
-      <joint name="joint_6">
-        <command_interface name="position">
-          <param name="min">{-2*pi}</param>
-          <param name="max">{2*pi}</param>
-        </command_interface>
-        <command_interface name="velocity"/>
-        <state_interface name="position">
-          <param name="initial_value">0.0</param>
-        </state_interface>
-        <state_interface name="velocity"/>
-      </joint>
+      <!-- 2. DOOSAN H2515 EKLEMLERİ (Sayısal sınırlar ile) -->
+      <xacro:macro name="doosan_joint_interface" params="name p_min p_max">
+        <joint name="${name}">
+          <command_interface name="position">
+            <param name="min">${p_min}</param>
+            <param name="max">${p_max}</param>
+          </command_interface>
+          <state_interface name="position">
+            <param name="initial_value">0.0</param>
+          </state_interface>
+          <state_interface name="velocity">
+            <param name="initial_value">0.0</param>
+          </state_interface>
+        </joint>
+      </xacro:macro>
+      <xacro:doosan_joint_interface name="joint_1" p_min="-6.28318" p_max="6.28318"/>
+      <xacro:doosan_joint_interface name="joint_2" p_min="-6.28318" p_max="6.28318"/>
+      <xacro:doosan_joint_interface name="joint_3" p_min="-3.14159" p_max="3.14159"/>
+      <xacro:doosan_joint_interface name="joint_4" p_min="-6.28318" p_max="6.28318"/>
+      <xacro:doosan_joint_interface name="joint_5" p_min="-6.28318" p_max="6.28318"/>
+      <xacro:doosan_joint_interface name="joint_6" p_min="-6.28318" p_max="6.28318"/>
     </ros2_control>
   </xacro:macro>

Commit message: carbody mesh

File: awi_description/urdf/cart_with_h2515.urdf.xacro (robot description, xacro)
@@ -4,10 +4,10 @@
   <xacro:arg name="sim_mode" default="true"/>
   <xacro:arg name="namespace" default=""/>
-  <!-- 1. KIZAK MEKANİK MODELİ -->
+  <xacro:arg name="component_name" default="right_front_fender"/>
   <link name="world"/>
   <link name="slideBar">
     <visual>
       <geometry>
-        <box size="30.0 0.2 0.1"/>
+        <box size="5.0 0.2 0.1"/>
       </geometry>
       <origin xyz="0 0 0" rpy="0 0 0"/>
@@ -21,4 +21,5 @@
     <inertial>
       <mass value="500.0"/>
+      <origin xyz="0 0 0" rpy="0 0 0"/>
       <inertia ixx="10.0" ixy="0.0" ixz="0.0" iyy="100.0" iyz="0.0" izz="100.0"/>
     </inertial>
@@ -56,8 +57,6 @@
     <dynamics damping="5.0" friction="1.0"/>
   </joint>
-  <!-- 2. DOOSAN H2515 GÖVDESİ -->
   <xacro:include filename="$(find awi_description)/xacro/macro.h2515.blue.xacro" />
   <xacro:h2515 namespace="$(arg namespace)"/>
-  <!-- 3. KART MONTAJI -->
   <joint name="cart_to_doosan_mount" type="fixed">
     <origin xyz="0 0 0.05" rpy="0 0 0"/>
@@ -65,8 +64,10 @@
     <child link="base_link"/>
   </joint>
-  <!-- 4. ROS2 CONTROL DONANIM KANALI -->
+  <xacro:include filename="$(find awi_description)/urdf/component.xacro" />
+  <xacro:car_component parent="world" component="$(arg component_name)">
+    <origin xyz="2.0 1.75 0.5" rpy="0 0 3.14159"/>
+  </xacro:car_component>
   <xacro:include filename="$(find awi_description)/urdf/inspection_cell_ros2_control.xacro" />
   <xacro:inspection_cell_ros2_control sim_mode="$(arg sim_mode)"/>
-  <!-- 5. TEK GAZEBO ROS2 CONTROL PLUGIN -->
   <gazebo>
     <plugin filename="ign_ros2_control-system" name="ign_ros2_control::IgnitionROS2ControlPlugin">
